File: motorthing-v2.brd (EAGLE design)
At the start: 42 x 42 mm, 16 parts, among them IC1 MAX485, IC2 4N25M, IC3 wemos D1 Mini, IC4 7805TV, J1 DCJ0202LARGE_VIA, X1 1501_0LARGE_VIA

Commit message: fix resistor values
Parts:
- R2: value 120 -> 1k
- R4: value 1k -> 120
Changed lines of the file:
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@@
 <attribute name="VALUE" x="39.37" y="16.51" size="1.27" layer="27" rot="R180"/>
 </element>
-<element name="R2" library="rcl" package="0207/10" value="120" x="20.32" y="20.32" rot="R180"/>
+<element name="R2" library="rcl" package="0207/10" value="1k" x="20.32" y="20.32" rot="R180"/>
 <element name="R3" library="rcl" package="0207/10" value="1k" x="13.97" y="30.48" rot="R90"/>
-<element name="R4" library="rcl" package="0207/10" value="1k" x="11.43" y="26.67" rot="R90"/>
+<element name="R4" library="rcl" package="0207/10" value="120" x="11.43" y="26.67" rot="R90"/>
 </elements>
 <signals>
